File: Hardware/PuppetSynth/PuppetSynth_v2_PCB.kicad_sch (KiCad schematic)
At the start: 48 parts, among them J1 ADS1115, J10 PINHD_1x16_Male, J11 JST_03, J12 JST_03, J13 JST_05, J14 JST_05, J15 JST_05, J16 JST_03, J17 JST_03, J18 JST_03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

Commit message: Updated PCBs, Archived 3D models, deleted old schematic
Parts:
- removed 10k3, 10k5, 10k7: R_Potentiometer, Potentiometer_THT:Potentiometer_Piher_T-16L_Single_Vertical_Hole, symbol Device:R_Potentiometer
- removed C1, C2, C6: 1uF, Capacitor_THT:C_Disc_D3.0mm_W2.0mm_P2.50mm, symbol PCM_SL_Devices:Capacitor_NP
- removed J10: PINHD_1x16_Male, Connector_PinHeader_2.54mm:PinHeader_2x08_P2.54mm_Vertical, symbol PCM_SL_Pin_Headers:PINHD_1x16_Male
- removed J19, J8: JST_05, Connector_JST:JST_EH_B5B-EH-A_1x05_P2.50mm_Vertical, symbol PCM_SL_Connectors:JST_05
- removed R15, R16, R19, R20, R7, R8: 2.2k, Resistor_THT:R_Axial_DIN0207_L6.3mm_D2.5mm_P10.16mm_Horizontal, symbol PCM_SL_Resistors:2.2k
- removed R18, R3, R6: 100ohm, Resistor_THT:R_Axial_DIN0207_L6.3mm_D2.5mm_P10.16mm_Horizontal, symbol PCM_SL_Resistors:2.2k
- removed SW1, SW4, SW6: SW_SP3T_NR01103, Button_Switch_THT:SW_NKK_NR01, symbol Switch:SW_SP3T_NR01103
- added C3, C4, C5: 1uF, Capacitor_THT:C_Disc_D3.0mm_W2.0mm_P2.50mm, symbol PCM_SL_Devices:Capacitor_NP
- added H1, H10, H11, H12, H13, H14, H15, H16, H17, H18, H2, H3, H4, H5, H6, H7, H8, H9: MountingHole_M3, MountingHole:MountingHole_3.2mm_M3, symbol PCM_SL_Mechanical:MountingHole_M3
- added J20, J21, J22, J24, J25, J26: JST_03, Connector_JST:JST_EH_B3B-EH-A_1x03_P2.50mm_Vertical, symbol PCM_SL_Connectors:JST_03
- added J8: PINHD_1x16_Male, Connector_PinHeader_2.54mm:PinHeader_2x08_P2.54mm_Vertical, symbol PCM_SL_Pin_Headers:PINHD_1x16_Male
- added R10, R11, R13, R14, R4, R5: 2.2k, Resistor_THT:R_Axial_DIN0207_L6.3mm_D2.5mm_P10.16mm_Horizontal, symbol PCM_SL_Resistors:2.2k
- added R12, R17, R9: 100ohm, Resistor_THT:R_Axial_DIN0207_L6.3mm_D2.5mm_P10.16mm_Horizontal, symbol PCM_SL_Resistors:2.2k
- 10k1, 10k2: footprint Potentiometer_THT:Potentiometer_Bourns_PTA6043_Single_Slide -> PuppetSynth:PS1001B1BR10K
- 10k4, 10k6, 10k8: footprint Potentiometer_THT:Potentiometer_Bourns_PTA6043_Single_Slide -> PuppetSynth:PS6020MC1BR10K
Connections:
- net +5V: now also J20.1, J21.1, J22.1, J8.16, R12.2, R17.2, R9.2
- net GND: now also C3.2, C4.2, C5.2, J20.3, J21.3, J22.3, J8.1, R10.1, R13.1, R5.1
- net 1 renamed Main_1
- net Main_1: now also J2.10, J8.15; no longer A1.9 (A0)
- net 10 renamed Small_Fader_2
- net Small_Fader_2: now also A1.13 (A4), J9.8, J8.8; no longer J2.10, J9.6
- net 11 renamed Small_Fader_3
- net Small_Fader_3: now also A1.10 (A1), J8.5; no longer A1.11 (A2)
- net 12 renamed Toggle_1
- net Toggle_1: now also A1.9 (A0), J8.4; no longer A1.12 (A3)
- net 13 renamed Toggle_2
- net Toggle_2: now also J1.7, C4.1, J25.2, J8.3; no longer A1.13 (A4)
- net 14 renamed Small_Fader_1
- net Small_Fader_1: now also 10k4.2, J13.2, J5.2, J9.11, J8.11; no longer J9.2
- net 2 renamed Main_2
- net Main_2: now also J2.9, J8.14; no longer A1.10 (A1)
- net 3 renamed Switch_1
- net Switch_1: now also J2.7, J8.13; no longer J1.7
- net 4 renamed Switch_2
- net Switch_2: now also J1.10, J9.10, J8.10; no longer J1.8, J9.12
- net 5 renamed Switch_3
- net Switch_3: now also J2.8, J9.7, J8.7; no longer J1.9, J9.11
- net 6 renamed Knob_1
- net Knob_1: now also J1.8, J9.12, J8.12; no longer J1.10, J9.10
- net 7 renamed Knob_2
- net Knob_2: now also J1.9, J21.2, J8.9; no longer J2.7
- net 8 renamed Knob_3
- net Knob_3: now also A1.11 (A2), J9.6, J22.2, J8.6; no longer J2.8, J9.8
- removed net 9: 10k4.2, J13.2, J2.9, J5.2, J9.7
- new net: C3.1, J24.2
- new net: J24.3, R4.1, R5.2
- new net: J24.1, R4.2, R9.1
- new net: J26.3, R13.2, R14.1
- new net: J26.1, R14.2, R17.1
- new net: J25.1, R11.2, R12.1
- new net: J25.3, R10.2, R11.1
- new net Toggle_3: A1.12 (A3), C5.1, J26.2, J8.2, J9.2
- no-connect marks 21 -> 20
Other:
- note added: "16 pin cable"
- note added: "Effect toggle resistors"
- note added: "Matching second prototype and code configuration. Change as needed"
- note added: "Mounting pins to reduce strain on PCBs and Faders. M3"
- note added: "to main faders"
- note added: "to smal faders, potentiometers and rotary switches"
- note removed: "Panel 3: Visual effect toggles - ON-OFF-ON momentary toggle switches"
- moved on the sheet: J11, J12, J13, J14, J15, J9

Commit message: updated pcb
Parts:
- removed H15, H16, H17, H18: MountingHole_M3, MountingHole:MountingHole_3.2mm_M3, symbol PCM_SL_Mechanical:MountingHole_M3
- removed J8, J9: PINHD_1x16_Male, Connector_PinHeader_2.54mm:PinHeader_2x08_P2.54mm_Vertical, symbol PCM_SL_Pin_Headers:PINHD_1x16_Male
- removed SW7: Switch, Button_Switch_THT:SW_SPST_Omron_B3F-40xx, symbol ScottoKeebs:Placeholder_Switch
Connections:
- no-connect marks 20 -> 21
Other:
- note added: "MCU - Arduino Leonardo - Pull-up resistors with bridged jumpers"
- note removed: "16 pin cable"
- note removed: "MCU - Arduino Leonardo - Pull-up resistors with bridged jumpers - Reset button"
- moved on the sheet: J1, J2
