File: Hardware/PuppetSynth/PuppetSynth_v2_PCB.kicad_pcb (KiCad board)
At the start: 2 copper layers, 406.4 x 343.1 mm, 48 parts, among them J1 ADS1115, J10 PINHD_1x16_Male, J11 JST_03, J12 JST_03, J13 JST_05, J14 JST_05, J15 JST_05, J16 JST_03, J17 JST_03, J18 JST_03, J19 JST_05, J2 ADS1115, J3 JST_03, J4 JST_03, J5 JST_05, J6 JST_05, J7 JST_05, J8 JST_05, J9 PINHD_1x16_Male, SW1 SW_SP3T_NR01103, SW4 SW_SP3T_NR01103, SW6 SW_SP3T_NR01103, SW7 Switch

Commit message: Updated PCBs, Archived 3D models, deleted old schematic
Parts:
- removed 10k3, 10k5, 10k7: R_Potentiometer, Potentiometer_THT:Potentiometer_Piher_T-16L_Single_Vertical_Hole
- removed C1, C2, C6: 1uF, Capacitor_THT:C_Disc_D3.0mm_W2.0mm_P2.50mm
- removed J10: PINHD_1x16_Male, Connector_PinHeader_2.54mm:PinHeader_2x08_P2.54mm_Vertical
- removed J19: JST_05, Connector_JST:JST_EH_B5B-EH-A_1x05_P2.50mm_Vertical
- removed R15, R16, R19, R20, R7, R8: 2.2k, Resistor_THT:R_Axial_DIN0207_L6.3mm_D2.5mm_P10.16mm_Horizontal
- removed R18, R3, R6: 100ohm, Resistor_THT:R_Axial_DIN0207_L6.3mm_D2.5mm_P10.16mm_Horizontal
- removed SW1, SW4, SW6: SW_SP3T_NR01103, Button_Switch_THT:SW_NKK_NR01
- added C3: 1uF, Capacitor_THT:C_Disc_D3.0mm_W2.0mm_P2.50mm, B.Cu at (359.4, 282.8)
- added C4: 1uF, Capacitor_THT:C_Disc_D3.0mm_W2.0mm_P2.50mm, B.Cu at (360.0, 270.1)
- added C5: 1uF, Capacitor_THT:C_Disc_D3.0mm_W2.0mm_P2.50mm, B.Cu at (360.0, 259.9)
- added H1: MountingHole_M3, MountingHole:MountingHole_3.2mm_M3, F.Cu at (229.0, 119.3)
- added H10: MountingHole_M3, MountingHole:MountingHole_3.2mm_M3, F.Cu at (321.0, 120.6)
- added H11: MountingHole_M3, MountingHole:MountingHole_3.2mm_M3, F.Cu at (338.8, 191.1)
- added H12: MountingHole_M3, MountingHole:MountingHole_3.2mm_M3, F.Cu at (321.0, 191.1)
- added H13: MountingHole_M3, MountingHole:MountingHole_3.2mm_M3, F.Cu at (269.0, 262.1)
- added H14: MountingHole_M3, MountingHole:MountingHole_3.2mm_M3, F.Cu at (427.1, 264.0)
- added H15: MountingHole_M3, MountingHole:MountingHole_3.2mm_M3, F.Cu at (389.0, 248.2)
- added H16: MountingHole_M3, MountingHole:MountingHole_3.2mm_M3, F.Cu at (389.7, 281.8)
- added H17: MountingHole_M3, MountingHole:MountingHole_3.2mm_M3, F.Cu at (306.5, 265.9)
- added H18: MountingHole_M3, MountingHole:MountingHole_3.2mm_M3, F.Cu at (351.6, 265.9)
- added H2: MountingHole_M3, MountingHole:MountingHole_3.2mm_M3, F.Cu at (248.0, 119.3)
- added H3: MountingHole_M3, MountingHole:MountingHole_3.2mm_M3, F.Cu at (229.0, 190.4)
- added H4: MountingHole_M3, MountingHole:MountingHole_3.2mm_M3, F.Cu at (248.0, 190.4)
- added H5: MountingHole_M3, MountingHole:MountingHole_3.2mm_M3, F.Cu at (274.0, 191.1)
- added H6: MountingHole_M3, MountingHole:MountingHole_3.2mm_M3, F.Cu at (291.8, 191.1)
- added H7: MountingHole_M3, MountingHole:MountingHole_3.2mm_M3, F.Cu at (292.5, 120.0)
- added H8: MountingHole_M3, MountingHole:MountingHole_3.2mm_M3, F.Cu at (274.0, 120.6)
- added H9: MountingHole_M3, MountingHole:MountingHole_3.2mm_M3, F.Cu at (338.8, 120.6)
- added J20: JST_03, Connector_JST:JST_EH_B3B-EH-A_1x03_P2.50mm_Vertical, B.Cu at (229.9, 112.4)
- added J21: JST_03, Connector_JST:JST_EH_B3B-EH-A_1x03_P2.50mm_Vertical, B.Cu at (287.5, 113.0)
- added J22: JST_03, Connector_JST:JST_EH_B3B-EH-A_1x03_P2.50mm_Vertical, B.Cu at (334.0, 113.6)
- added J24: JST_03, Connector_JST:JST_EH_B3B-EH-A_1x03_P2.50mm_Vertical, B.Cu at (377.7, 249.8)
- added J25: JST_03, Connector_JST:JST_EH_B3B-EH-A_1x03_P2.50mm_Vertical, B.Cu at (377.7, 262.5)
- added J26: JST_03, Connector_JST:JST_EH_B3B-EH-A_1x03_P2.50mm_Vertical, B.Cu at (377.7, 275.2)
- added R10: 2.2k, Resistor_THT:R_Axial_DIN0207_L6.3mm_D2.5mm_P10.16mm_Horizontal, B.Cu at (372.7, 261.5)
- added R11: 2.2k, Resistor_THT:R_Axial_DIN0207_L6.3mm_D2.5mm_P10.16mm_Horizontal, B.Cu at (372.7, 265.6)
- added R12: 100ohm, Resistor_THT:R_Axial_DIN0207_L6.3mm_D2.5mm_P10.16mm_Horizontal, B.Cu at (372.7, 269.6)
- added R13: 2.2k, Resistor_THT:R_Axial_DIN0207_L6.3mm_D2.5mm_P10.16mm_Horizontal, B.Cu at (372.7, 273.7)
- added R14: 2.2k, Resistor_THT:R_Axial_DIN0207_L6.3mm_D2.5mm_P10.16mm_Horizontal, B.Cu at (372.7, 277.7)
- added R17: 100ohm, Resistor_THT:R_Axial_DIN0207_L6.3mm_D2.5mm_P10.16mm_Horizontal, B.Cu at (372.7, 281.8)
- added R4: 2.2k, Resistor_THT:R_Axial_DIN0207_L6.3mm_D2.5mm_P10.16mm_Horizontal, B.Cu at (372.7, 249.4)
- added R5: 2.2k, Resistor_THT:R_Axial_DIN0207_L6.3mm_D2.5mm_P10.16mm_Horizontal, B.Cu at (372.7, 253.4)
- added R9: 100ohm, Resistor_THT:R_Axial_DIN0207_L6.3mm_D2.5mm_P10.16mm_Horizontal, B.Cu at (372.7, 257.5)
- 10k1, 10k2: footprint Potentiometer_THT:Potentiometer_Bourns_PTA6043_Single_Slide -> PuppetSynth:PS1001B1BR10K
- 10k4, 10k6, 10k8: footprint Potentiometer_THT:Potentiometer_Bourns_PTA6043_Single_Slide -> PuppetSynth:PS6020MC1BR10K
- J8: value JST_05 -> PINHD_1x16_Male; footprint Connector_JST:JST_EH_B5B-EH-A_1x05_P2.50mm_Vertical -> Connector_PinHeader_2.54mm:PinHeader_2x08_P2.54mm_Vertical; moved to F.Cu
- moved 10k1 162.5 mm to (263.1, 263.7), turned to 180 degrees
- moved J3 95.3 mm to (275.1, 259.6)
- moved J16 62.7 mm to (242.9, 112.5)
- moved J8 56.6 mm to (343.8, 360.6), turned to -90 degrees
- moved J18 53.6 mm to (320.6, 113.6)
- moved J14 53.0 mm to (325.4, 258.3)
- moved J15 53.0 mm to (307.7, 258.3)
- moved J13 53.0 mm to (343.0, 258.3)
- moved J9 50.3 mm to (337.1, 276.7)
- moved J17 50.2 mm to (274.1, 113.0)
- moved J12 49.9 mm to (306.6, 277.3)
- moved J11 49.1 mm to (351.4, 272.3)
- moved A1 43.6 mm to (352.2, 337.7)
- moved J1 43.6 mm to (323.0, 353.0)
- moved J2 43.6 mm to (345.9, 370.7)
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Connections:
- 10k1 pad 2: 1 -> Main_1
- 10k2 pad 2: 2 -> Main_2
- A1 pad 10: 2 -> Small_Fader_3
- A1 pad 11: 11 -> Knob_3
- A1 pad 12: 12 -> Toggle_3
- A1 pad 13: 13 -> Small_Fader_2
- A1 pad 14: 14 -> Small_Fader_1
- A1 pad 9: 1 -> Toggle_1
- J1 pad 10: 6 -> Switch_2
- J1 pad 7: 3 -> Toggle_2
- J1 pad 8: 4 -> Knob_1
- J1 pad 9: 5 -> Knob_2
- J11 pad 2: 1 -> Main_1
- J12 pad 2: 2 -> Main_2
- J13 pad 2: 9 -> Small_Fader_1
- J13 pad 3: 6 -> Knob_1
- J13 pad 4: 3 -> Switch_1
- J14 pad 2: 10 -> Small_Fader_2
- J14 pad 3: 7 -> Knob_2
- J14 pad 4: 4 -> Switch_2
- J15 pad 2: 11 -> Small_Fader_3
- J15 pad 3: 8 -> Knob_3
- J15 pad 4: 5 -> Switch_3
- J16 pad 2: 3 -> Switch_1
- J17 pad 2: 4 -> Switch_2
- J18 pad 2: 5 -> Switch_3
- J2 pad 10: 10 -> Main_1
- J2 pad 7: 7 -> Switch_1
- J2 pad 8: 8 -> Switch_3
- J2 pad 9: 9 -> Main_2
- J3 pad 2: 1 -> Main_1
- J4 pad 2: 2 -> Main_2
- J5 pad 2: 9 -> Small_Fader_1
- J5 pad 3: 6 -> Knob_1
- J5 pad 4: 3 -> Switch_1
- J6 pad 2: 10 -> Small_Fader_2
- J6 pad 3: 7 -> Knob_2
- J6 pad 4: 4 -> Switch_2
- J7 pad 2: 11 -> Small_Fader_3
- J7 pad 3: 8 -> Knob_3
- J7 pad 4: 5 -> Switch_3
- J8 pad 2: 14 -> Toggle_3
- J8 pad 3: 13 -> Toggle_2
- J8 pad 4: 12 -> Toggle_1
- J8 pad 5: +5V -> Small_Fader_3
- J9 pad 10: 6 -> Switch_2
- J9 pad 11: 5 -> Small_Fader_1
- J9 pad 12: 4 -> Knob_1
- J9 pad 13: 3 -> Switch_1
- J9 pad 14: 2 -> Main_2
- J9 pad 15: 1 -> Main_1
- J9 pad 2: 14 -> Toggle_3
- J9 pad 3: 13 -> Toggle_2
- J9 pad 4: 12 -> Toggle_1
- J9 pad 5: 11 -> Small_Fader_3
- J9 pad 6: 10 -> Knob_3
- J9 pad 7: 9 -> Switch_3
- J9 pad 8: 8 -> Small_Fader_2
- J9 pad 9: 7 -> Knob_2
Other:
- board size 406.4 x 343.1 mm -> 435.3 x 289.1 mm
- board text added: "5V Effect 1 GND"
- board text added: "5V Effect 2 GND"
- board text added: "5V Effect 3 GND"
- board text added: "5V Knob GND"
- board text removed: "5V 1 2 3 GND"
- board text removed: "5V Effect 1 Effect 2 Effect 3 GND"
- board text removed: "FX"
- board text removed: "FX 1"
- board text removed: "FX 2"
- board text removed: "FX 3"

Commit message: updated pcb
Parts:
- removed H15, H16, H17, H18: MountingHole_M3, MountingHole:MountingHole_3.2mm_M3
- removed J8, J9: PINHD_1x16_Male, Connector_PinHeader_2.54mm:PinHeader_2x08_P2.54mm_Vertical
- removed SW7: Switch, Button_Switch_THT:SW_SPST_Omron_B3F-40xx
- A1: footprint Module:Arduino_UNO_R3 -> Module:Arduino_UNO_R3_WithMountingHoles; moved to F.Cu
- moved R5 107.4 mm to (329.6, 351.8), turned to 90 degrees
- moved R4 100.5 mm to (332.7, 341.6), turned to -90 degrees
- moved R9 96.0 mm to (326.4, 341.6), turned to -90 degrees
- moved R10 95.6 mm to (341.0, 351.8), turned to 90 degrees
- moved C5 90.3 mm to (349.5, 349.6), turned to -135 degrees
- moved R11 81.2 mm to (344.2, 341.6), turned to -90 degrees
- moved R12 80.0 mm to (337.8, 341.6), turned to -90 degrees
- moved R13 79.1 mm to (360.0, 351.8), turned to 90 degrees
- moved C4 76.5 mm to (349.5, 345.8), turned to -135 degrees
- moved J24 74.4 mm to (344.9, 316.5), turned to 0 degrees
- moved J25 71.0 mm to (344.9, 325.4), turned to 0 degrees
- moved J26 67.7 mm to (344.8, 334.3), turned to 0 degrees
- moved R14 65.8 mm to (356.9, 341.6), turned to -90 degrees
- moved H14 65.2 mm to (429.8, 329.2)
- moved J4 65.2 mm to (424.1, 331.9)
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Connections:
- A1 pad 3: Net-(A1-~{RESET}) -> unconnected-(A1-~{RESET}-Pad3)
Routing:
- net +5V: track 0.00 -> 148.7 mm
- net SCL: track 0.00 -> 66.2 mm
- net SDA: track 0.00 -> 61.7 mm
- net Net-(J24-Pad1): track 0.00 -> 51.8 mm
- net Main_1: track 0.00 -> 43.2 mm
- net Switch_2: track 0.00 -> 39.9 mm
- net Knob_2: track 0.00 -> 39.2 mm
- net Net-(J24-Pad3): track 0.00 -> 38.0 mm
- net Small_Fader_1: track 0.00 -> 35.8 mm, vias 0 -> 1
- net Toggle_2: track 0.00 -> 33.7 mm
- net Switch_3: track 0.00 -> 32.9 mm
- net Net-(J25-Pad1): track 0.00 -> 31.9 mm
- net Knob_1: track 0.00 -> 29.1 mm
- net Knob_3: track 0.00 -> 28.3 mm
- net Net-(C3-Pad1): track 0.00 -> 28.1 mm
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- added copper zone on B.Cu, net GND
- added copper zone on F.Cu, net GND
Other:
- board size 435.3 x 289.1 mm -> 445.2 x 254.9 mm
- board text added: "3"
- board text added: "4"
- board text added: "5"
- board text added: "ADS1115"
- board text added: "Effect 1"
- board text added: "Effect 2"
- board text added: "Effect 3"
- board text removed: "5V Effect 1 GND"
- board text removed: "5V Effect 2 GND"
- board text removed: "5V Effect 3 GND"

Commit message: updated pcb
Parts:
- removed J1, J2: ADS1115, Connector_PinSocket_2.54mm:PinSocket_1x10_P2.54mm_Vertical
- removed the JP2 at (364.5, 337.2)
- added G***: LOGO, LOGO, F.Cu at (347.9, 329.6)
- added G***: LOGO, LOGO, F.Cu at (347.7, 319.7)
- added G***: LOGO, LOGO, B.Cu at (326.1, 346.5)
- added J10: PINHD_1x6_Female, Connector_PinSocket_2.54mm:PinSocket_1x06_P2.54mm_Vertical, B.Cu at (367.2, 336.6)
- added J19: PINHD_1x6_Female, Connector_PinSocket_2.54mm:PinSocket_1x06_P2.54mm_Vertical, B.Cu at (367.2, 323.9)
- added J8: PINHD_1x6_Female, Connector_PinSocket_2.54mm:PinSocket_1x06_P2.54mm_Vertical, B.Cu at (340.4, 336.2)
- added J9: PINHD_1x6_Female, Connector_PinSocket_2.54mm:PinSocket_1x06_P2.54mm_Vertical, B.Cu at (340.1, 323.7)
- added JP2: Jumper_2_Bridged, Jumper:SolderJumper-2_P1.3mm_Open_RoundedPad1.0x1.5mm, B.Cu at (367.6, 328.2)
- added JP2: Jumper_2_Bridged, Jumper:SolderJumper-2_P1.3mm_Open_RoundedPad1.0x1.5mm, B.Cu at (333.7, 336.2)
- A1: footprint Module:Arduino_UNO_R3_WithMountingHoles -> Module:Arduino_UNO_R3
- moved J26 32.4 mm to (330.9, 305.1)
- moved J25 30.1 mm to (331.0, 298.7)
- moved J24 27.9 mm to (331.0, 292.4)
- moved J12 21.6 mm to (346.6, 315.1), turned to 0 degrees
- moved J11 20.0 mm to (360.8, 315.2), turned to 0 degrees
- moved J13 18.7 mm to (361.9, 305.1), turned to 90 degrees
- moved C3 14.9 mm to (364.4, 341.8)
- moved C4 14.7 mm to (364.2, 345.7)
- moved C5 14.6 mm to (364.1, 349.6)
- moved J14 12.3 mm to (355.3, 305.1), turned to 90 degrees
- moved J15 11.5 mm to (348.6, 305.0), turned to 90 degrees
- moved R4 7.13 mm to (339.9, 341.1)
- moved R5 7.00 mm to (336.6, 351.3)
- moved R9 6.88 mm to (333.2, 341.1)
- moved JP1 6.25 mm to (367.6, 331.0), turned to 180 degrees
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Routing:
- net +5V: track 148.7 -> 0.00 mm
- net SCL: track 66.2 -> 0.00 mm
- net SDA: track 61.7 -> 0.00 mm
- net Net-(J24-Pad1): track 51.8 -> 0.00 mm
- net Main_1: track 43.2 -> 0.00 mm
- net Switch_2: track 39.9 -> 0.00 mm
- net Knob_2: track 39.2 -> 0.00 mm
- net Net-(J24-Pad3): track 38.0 -> 0.00 mm
- net Small_Fader_1: track 35.8 -> 0.00 mm, vias 1 -> 0
- net Toggle_2: track 33.7 -> 0.00 mm
- net Switch_3: track 32.9 -> 0.00 mm
- net Net-(J25-Pad1): track 31.9 -> 0.00 mm
- net Knob_1: track 29.1 -> 0.00 mm
- net Knob_3: track 28.3 -> 0.00 mm
- net Net-(C3-Pad1): track 28.1 -> 0.00 mm
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Other:
- board text added: "16-bit ADC"
- board text added: "A+"
- board text added: "A-"
- board text added: "A0"
- board text added: "A1"
- board text added: "A2"
- board text added: "A3"
- board text added: "ADDR"
- board text added: "ALRT"
- board text added: "FX3 FX2 FX1"
- board text added: "GND"
- board text added: "Main 1"
- board text added: "Main 2"
- board text added: "PUPPET SYNTHESIZER PCB by Silvan Roth ZHdK 2025"
- board text added: "Repo"
- board text added: "SCL"
- board text added: "SDA"
- board text added: "VIN"
- board text added: "Wave 1 Wave 2 Wave 3"
- board text removed: "1"
- board text removed: "2"
- board text removed: "3"
- board text removed: "4"
- board text removed: "5"
- board text removed: "Effect 1"
- board text removed: "Effect 2"
- board text removed: "Effect 3"
- board text removed: "SDA SCL"

Commit message: updated pcb
Parts:
- removed the JP2 at (333.7, 336.2)
- JP1, JP2: moved to F.Cu
- moved R13 13.0 mm to (346.3, 351.3)
- moved R12 9.78 mm to (352.9, 341.1)
- moved R17 9.78 mm to (343.2, 341.1)
- moved R10 9.78 mm to (356.1, 351.3)
- moved R11 9.78 mm to (359.3, 341.1)
- moved R14 6.60 mm to (349.5, 341.1)
- turned JP1 to 0 degrees
- turned JP2 to 0 degrees
Connections:
- J19 pad 2: unconnected-(J19-Pad2) -> Main_1
- J19 pad 3: Main_1 -> Main_2
- J19 pad 4: Main_2 -> Switch_3
- J19 pad 5: Switch_3 -> Switch_1
- J19 pad 6: Switch_1 -> unconnected-(J19-Pad6)
Routing:
- net +5V: track 0.00 -> 260.1 mm
- net GND: track 0.00 -> 240.4 mm
- net Switch_3: track 0.00 -> 117.8 mm, vias 0 -> 1
- net Knob_3: track 0.00 -> 115.5 mm
- net Net-(C3-Pad1): track 0.00 -> 83.8 mm
- net Net-(J25-Pad3): track 0.00 -> 79.0 mm
- net Toggle_2: track 0.00 -> 74.8 mm
- net Toggle_3: track 0.00 -> 73.1 mm
- net Net-(J24-Pad1): track 0.00 -> 69.9 mm
- net Net-(J24-Pad3): track 0.00 -> 67.1 mm
- net Small_Fader_1: track 0.00 -> 56.5 mm, vias 0 -> 1
- net Net-(J26-Pad3): track 0.00 -> 48.9 mm, vias 0 -> 1
- net Knob_1: track 0.00 -> 48.5 mm, vias 0 -> 2
- net Small_Fader_2: track 0.00 -> 41.0 mm
- net Knob_2: track 0.00 -> 36.5 mm
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
Commit message: updated PCB: Rounded traces and shield edges
Parts:
- moved G*** 0.90 mm to (347.7, 328.7)
- moved G*** 0.25 mm to (325.9, 346.5)
Routing:
- net Net-(J25-Pad3): track 79.0 -> 77.1 mm
- net Toggle_3: track 73.1 -> 71.4 mm
- net Toggle_2: track 74.8 -> 73.3 mm
- net Net-(C3-Pad1): track 83.8 -> 82.4 mm
- net Switch_3: track 117.8 -> 116.5 mm
- net Net-(J24-Pad3): track 67.1 -> 65.9 mm
- net Knob_3: track 115.5 -> 114.4 mm
- net Net-(J24-Pad1): track 69.9 -> 68.9 mm
- net Small_Fader_1: track 56.5 -> 55.5 mm
- net Knob_2: track 36.5 -> 35.6 mm
- net Knob_1: track 48.5 -> 47.5 mm
- net Net-(J26-Pad3): track 48.9 -> 48.1 mm
- net Switch_1: track 33.7 -> 32.9 mm
- net Small_Fader_3: track 31.2 -> 30.4 mm
- net GND: track 240.4 -> 239.7 mm
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Other:
- outline, holes or cut-outs redrawn

Commit message: Updated schematic and PCB
fixed symbols in schematic, rearranged some parts on PCB, ran traces, aesthetic improvements, fixed layers
Parts:
- removed 10k2: R_Potentiometer, PuppetSynth:PS1001B1BR10K
- removed 10k6, 10k8: R_Potentiometer, PuppetSynth:PS6020MC1BR10K
- removed H10, H11, H12, H14, H5, H6, H7, H8, H9: MountingHole_M3, MountingHole:MountingHole_3.2mm_M3
- removed J17, J18, J21, J22, J4: JST_03, Connector_JST:JST_EH_B3B-EH-A_1x03_P2.50mm_Vertical
- removed J6, J7: JST_05, Connector_JST:JST_EH_B5B-EH-A_1x05_P2.50mm_Vertical
- moved C3 347.6 mm to (192.0, 39.9), turned to -90 degrees
- moved C4 345.7 mm to (192.0, 46.0), turned to -90 degrees
- moved C5 343.7 mm to (192.0, 52.1), turned to -90 degrees
- moved J13 285.5 mm to (226.8, 53.7)
- moved A1 285.5 mm to (188.1, 74.9)
- moved G*** 285.5 mm to (212.6, 68.2)
- moved J10 285.5 mm to (232.0, 85.1)
- moved J11 285.5 mm to (225.6, 63.7)
- moved J14 285.5 mm to (220.2, 53.6)
- moved J19 285.5 mm to (232.0, 72.4)
- moved J8 285.5 mm to (205.2, 84.7)
- moved J9 285.5 mm to (205.0, 72.2)
- moved JP1 285.5 mm to (232.5, 79.5)
- moved JP2 285.5 mm to (232.5, 76.7)
- moved R1 285.5 mm to (236.0, 89.6)
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- renumbered 10k4 to 10k, 10k1 to 10k
Connections:
- J20 pad 2: unconnected-(J20-Pad2) -> Knob_1
Routing:
- net GND: track 239.7 -> 0.00 mm, vias 0 -> 6
- net Knob_1: track 47.5 -> 142.1 mm, vias 2 -> 0
- net Switch_1: track 32.9 -> 116.1 mm
- net Knob_3: track 114.4 -> 32.5 mm
- net Switch_3: track 116.5 -> 40.4 mm, vias 1 -> 0
- net Net-(C3-Pad1): track 82.4 -> 9.43 mm
- net Net-(J25-Pad1): track 12.6 -> 71.1 mm, vias 0 -> 1
- net Toggle_3: track 71.4 -> 18.8 mm
- net Net-(J26-Pad1): track 12.6 -> 55.5 mm, vias 0 -> 1
- net Toggle_2: track 73.3 -> 39.8 mm
- net SDA: track 35.1 -> 61.2 mm
- net SCL: track 34.4 -> 53.9 mm
- net Main_1: track 9.49 -> 27.9 mm
- net Net-(J25-Pad3): track 77.1 -> 62.4 mm, vias 0 -> 1
- net Main_2: track 31.3 -> 20.8 mm
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Other:
- board size 445.2 x 254.9 mm -> 166.8 x 155.2 mm
- board text added: "5V"
- board text added: "Analog in"
- board text added: "SDA SCL"
- board text removed: "A+"
- board text removed: "A-"
